File: 65Numpad.sch (KiCad schematic (older format))
At the start: 180 parts, among them J1 MX-NoLED, K1 MX-NoLED, M1 MX-NoLED, P1 MX-NoLED, Q1 MX-NoLED, T1 MX-NoLED, U2 MX-NoLED, X1 MX-NoLED, Y1 MX-NoLED

Commit message: Schematic 1u addons
Parts:
- added ALTENTER1, ALTPLUS1, ALTZERO1: MX-NoLED, MX_Only:MXOnly-2U-ReversedStabilizers-NoLEDHotSwap, symbol MX_Alps_Hybrid:MX-NoLED
- added OPTION2, OPTION5, OPTION6: MX-NoLED, MX_Only:MXOnly-1U-NoLEDHotswap, symbol MX_Alps_Hybrid:MX-NoLED
- ENTER2, PLUS1, ZERO2: footprint MX_Only:MXOnly-2U-NoLEDHotswap -> MX_Only:MXOnly-2U-ReversedStabilizers-NoLEDHotSwap
- SPACE1: footprint MX_Only:MXOnly-6.25U-NoLEDHotswap -> MX_Only:MXOnly-6.25U-ReversedStabilizers-NoLEDHotswap
- renumbered OPTION2 to OPTION3, OPTION3 to OPTION4
Connections:
- net COL1: no longer D30.1 (K), D32.1 (K), D34.1 (K), D36.1 (K), D38.1 (K), D40.1 (K), D42.1 (K), D83.1 (K), D84.1 (K), D85.1 (K), Main1.14 (16/PB2), Numpad1.10 (7/PE6)
- net COL3: now also ALTENTER1.1 (COL), ALTPLUS1.1 (COL), ALTZERO1.1 (COL), OPTION5.1 (COL), OPTION6.1 (COL); no longer D10.1 (K), D12.1 (K), D14.1 (K), D15.1 (K), D16.1 (K), D17.1 (K), D18.1 (K), D19.1 (K), D2.1 (K), D20.1 (K), D21.1 (K), D22.1 (K), D23.1 (K), D24.1 (K), D25.1 (K), D26.1 (K), D27.1 (K), D28.1 (K), D4.1 (K), D6.1 (K), D73.1 (K), D74.1 (K), D75.1 (K), D76.1 (K), D77.1 (K), D78.1 (K), D79.1 (K), D8.1 (K), D80.1 (K), D81.1 (K), D82.1 (K), D86.1 (K), D87.1 (K), Main1.16 (15/PB1), Main1.17 (A0/PF7), Main1.18 (A1/PF6), Numpad1.7 (4/PD4), Numpad1.8 (5/PC6), Numpad1.9 (6/PD7)
- net at D79.2 (A), PLUS1.2 (ROW): now also OPTION2.2 (ROW)
- net at D85.2 (A), ENTER2.2 (ROW): now also ALTZERO1.2 (ROW), OPTION5.2 (ROW), OPTION6.2 (ROW)
- net at D86.2 (A), OPTION1.2 (ROW): now also ALTPLUS1.2 (ROW)
- net at D87.2 (A), OPTION3.2 (ROW): now also ALTENTER1.2 (ROW)
- net ROW4: now reaches D88.1 (K)
- net ROW4: now also D30.1 (K), D32.1 (K), D34.1 (K), D36.1 (K), D38.1 (K), D40.1 (K), D42.1 (K), D83.1 (K), D84.1 (K), D85.1 (K), Main1.14 (16/PB2), Numpad1.10 (7/PE6)
- new net ROW1: D10.1 (K), D12.1 (K), D14.1 (K), D2.1 (K), D4.1 (K), D6.1 (K), D73.1 (K), D74.1 (K), D75.1 (K), D8.1 (K), D86.1 (K), Main1.18 (A1/PF6), Numpad1.7 (4/PD4)
- new net ROW2: D15.1 (K), D17.1 (K), D19.1 (K), D21.1 (K), D23.1 (K), D25.1 (K), D27.1 (K), D76.1 (K), D77.1 (K), D78.1 (K), D79.1 (K), Main1.17 (A0/PF7), Numpad1.8 (5/PC6)
- new net ROW3: D16.1 (K), D18.1 (K), D20.1 (K), D22.1 (K), D24.1 (K), D26.1 (K), D28.1 (K), D80.1 (K), D81.1 (K), D82.1 (K), D87.1 (K), Main1.16 (15/PB1), Numpad1.9 (6/PD7)
Changed lines of the file:
@@
 F 0 "SPACE1" H 5283 5773 60  0000 C CNN
 F 1 "MX-NoLED" H 5283 5699 20  0000 C CNN
-F 2 "MX_Only:MXOnly-6.25U-NoLEDHotswap" H 4625 5525 60  0001 C CNN
+F 2 "MX_Only:MXOnly-6.25U-ReversedStabilizers-NoLEDHotswap" H 4625 5525 60  0001 C CNN
 F 3 "" H 4625 5525 60  0001 C CNN
 	1    5250 5550
@@
 F 0 "ZERO2" H 15283 5373 60  0000 C CNN
 F 1 "MX-NoLED" H 15283 5299 20  0000 C CNN
-F 2 "MX_Only:MXOnly-2U-NoLEDHotswap" H 14625 5125 60  0001 C CNN
+F 2 "MX_Only:MXOnly-2U-ReversedStabilizers-NoLEDHotSwap" H 14625 5125 60  0001 C CNN
 F 3 "" H 14625 5125 60  0001 C CNN
 	1    15250 5150
@@
 F 0 "PLUS1" H 16833 3823 60  0000 C CNN
 F 1 "MX-NoLED" H 16833 3749 20  0000 C CNN
-F 2 "MX_Only:MXOnly-2U-NoLEDHotswap" H 16175 3575 60  0001 C CNN
+F 2 "MX_Only:MXOnly-2U-ReversedStabilizers-NoLEDHotSwap" H 16175 3575 60  0001 C CNN
 F 3 "" H 16175 3575 60  0001 C CNN
 	1    16800 3600
@@
 F 0 "ENTER2" H 16833 5373 60  0000 C CNN
 F 1 "MX-NoLED" H 16833 5299 20  0000 C CNN
-F 2 "MX_Only:MXOnly-2U-NoLEDHotswap" H 16175 5125 60  0001 C CNN
+F 2 "MX_Only:MXOnly-2U-ReversedStabilizers-NoLEDHotSwap" H 16175 5125 60  0001 C CNN
 F 3 "" H 16175 5125 60  0001 C CNN
 	1    16800 5150
@@
 Connection ~ 16100 5600
 Wire Wire Line
-	16100 5600 15950 5600
-Wire Wire Line
 	15400 5100 15400 4350
 Connection ~ 15400 2050
@@
 	16950 1800 16950 2050
 Connection ~ 16950 2050
-Wire Wire Line
-	16950 2050 16950 2800
 Connection ~ 16950 3550
-Wire Wire Line
-	16950 3550 16950 4050
 Text GLabel 14850 2550 0    50   Input ~ 0
 ROW0
@@
 $EndComp
 $Comp
-L MX_Alps_Hybrid:MX-NoLED OPTION2
+L MX_Alps_Hybrid:MX-NoLED OPTION3
 U 1 1 60172190
 P 16800 4400
-AR Path="/60172190" Ref="OPTION2"  Part="1"
+AR Path="/60172190" Ref="OPTION3"  Part="1"
 AR Path="/6009603F/60172190" Ref="OPTION?"  Part="1"
-F 0 "OPTION2" H 16833 4623 60  0000 C CNN
+F 0 "OPTION3" H 16833 4623 60  0000 C CNN
 F 1 "MX-NoLED" H 16833 4549 20  0000 C CNN
 F 2 "MX_Only:MXOnly-1U-NoLEDHotswap" H 16175 4375 60  0001 C CNN
@@
 $EndComp
 $Comp
-L MX_Alps_Hybrid:MX-NoLED OPTION3
+L MX_Alps_Hybrid:MX-NoLED OPTION4
 U 1 1 6019024A
 P 15800 5150
-AR Path="/6019024A" Ref="OPTION3"  Part="1"
+AR Path="/6019024A" Ref="OPTION4"  Part="1"
 AR Path="/6009603F/6019024A" Ref="OPTION?"  Part="1"
-F 0 "OPTION3" H 15833 5373 60  0000 C CNN
+F 0 "OPTION4" H 15833 5373 60  0000 C CNN
 F 1 "MX-NoLED" H 15833 5299 20  0000 C CNN
 F 2 "MX_Only:MXOnly-1U-NoLEDHotswap" H 15175 5125 60  0001 C CNN
@@
 	15950 4350 15950 5100
 Connection ~ 15950 4350
-Connection ~ 15950 5600
-Wire Wire Line
-	15950 5600 15050 5600
-Connection ~ 15950 5100
-Wire Wire Line
-	15950 5100 15950 5600
 Wire Wire Line
 	16100 4850 16600 4850
 Connection ~ 16100 4850
-Connection ~ 16950 4850
-Wire Wire Line
-	16950 4850 16950 5100
-Connection ~ 16600 4850
-Wire Wire Line
-	16600 4850 16950 4850
 Wire Wire Line
 	16100 3300 16600 3300
 Connection ~ 16100 3300
-Connection ~ 16950 3300
-Wire Wire Line
-	16950 3300 16950 3550
-Connection ~ 16600 3300
-Wire Wire Line
-	16600 3300 16950 3300
 Connection ~ 16950 2800
-Wire Wire Line
-	16950 2800 16950 3300
 Connection ~ 16950 4350
-Wire Wire Line
-	16950 4350 16950 4850
-Wire Wire Line
-	16600 4050 16950 4050
-Connection ~ 16600 4050
-Connection ~ 16950 4050
-Wire Wire Line
-	16950 4050 16950 4350
+Connection ~ 15600 5600
+Wire Wire Line
+	15600 5600 15050 5600
+Wire Wire Line
+	15600 5600 16100 5600
+Wire Wire Line
+	16950 3550 16950 4250
+Wire Wire Line
+	16950 4350 16950 5000
+Wire Wire Line
+	16950 2800 16950 3550
+$Comp
+L MX_Alps_Hybrid:MX-NoLED ALTPLUS1
+U 1 1 601ED11B
+P 17300 2850
+AR Path="/601ED11B" Ref="ALTPLUS1"  Part="1"
+AR Path="/6009603F/601ED11B" Ref="OPTION?"  Part="1"
+F 0 "ALTPLUS1" H 17333 3073 60  0000 C CNN
+F 1 "MX-NoLED" H 17333 2999 20  0000 C CNN
+F 2 "MX_Only:MXOnly-2U-ReversedStabilizers-NoLEDHotSwap" H 16675 2825 60  0001 C CNN
+F 3 "" H 16675 2825 60  0001 C CNN
+	1    17300 2850
+	1    0    0    -1
+$EndComp
+Wire Wire Line
+	16950 2050 16950 2700
+Wire Wire Line
+	16750 3000 17250 3000
+Connection ~ 16750 3000
+Wire Wire Line
+	17450 2800 17450 2700
+Wire Wire Line
+	17450 2700 16950 2700
+Connection ~ 16950 2700
+Wire Wire Line
+	16950 2700 16950 2800
+$Comp
+L MX_Alps_Hybrid:MX-NoLED ALTZERO1
+U 1 1 6031C7B4
+P 17300 5150
+AR Path="/6031C7B4" Ref="ALTZERO1"  Part="1"
+AR Path="/6009603F/6031C7B4" Ref="ALTPLUS?"  Part="1"
+F 0 "ALTZERO1" H 17333 5373 60  0000 C CNN
+F 1 "MX-NoLED" H 17333 5299 20  0000 C CNN
+F 2 "MX_Only:MXOnly-2U-ReversedStabilizers-NoLEDHotSwap" H 16675 5125 60  0001 C CNN
+F 3 "" H 16675 5125 60  0001 C CNN
+	1    17300 5150
+	1    0    0    -1
+$EndComp
+Wire Wire Line
+	16750 5300 17250 5300
+Wire Wire Line
+	17450 5100 17450 5000
+Wire Wire Line
+	17450 5000 16950 5000
+Connection ~ 16950 5000
+Wire Wire Line
+	16950 5000 16950 5100
+Connection ~ 16750 5300
+$Comp
+L MX_Alps_Hybrid:MX-NoLED ALTENTER1
+U 1 1 6034204C
+P 17300 4400
+AR Path="/6034204C" Ref="ALTENTER1"  Part="1"
+AR Path="/6009603F/6034204C" Ref="ALTPLUS?"  Part="1"
+F 0 "ALTENTER1" H 17333 4623 60  0000 C CNN
+F 1 "MX-NoLED" H 17333 4549 20  0000 C CNN
+F 2 "MX_Only:MXOnly-2U-ReversedStabilizers-NoLEDHotSwap" H 16675 4375 60  0001 C CNN
+F 3 "" H 16675 4375 60  0001 C CNN
+	1    17300 4400
+	1    0    0    -1
+$EndComp
+Wire Wire Line
+	16750 4550 17250 4550
+Wire Wire Line
+	17450 4350 17450 4250
+Wire Wire Line
+	17450 4250 16950 4250
+Connection ~ 16950 4250
+Wire Wire Line
+	16950 4250 16950 4350
+Connection ~ 16750 4550
+$Comp
+L MX_Alps_Hybrid:MX-NoLED OPTION5
+U 1 1 603B6F36
+P 17800 5150
+AR Path="/603B6F36" Ref="OPTION5"  Part="1"
+AR Path="/6009603F/603B6F36" Ref="ALTPLUS?"  Part="1"
+F 0 "OPTION5" H 17833 5373 60  0000 C CNN
+F 1 "MX-NoLED" H 17833 5299 20  0000 C CNN
+F 2 "MX_Only:MXOnly-1U-NoLEDHotswap" H 17175 5125 60  0001 C CNN
+F 3 "" H 17175 5125 60  0001 C CNN
+	1    17800 5150
+	1    0    0    -1
+$EndComp
+Wire Wire Line
+	17250 5300 17750 5300
+Wire Wire Line
+	17950 5100 17950 5000
+Wire Wire Line
+	17950 5000 17450 5000
+$Comp
+L MX_Alps_Hybrid:MX-NoLED OPTION6
+U 1 1 603D70FA
+P 18300 5150
+AR Path="/603D70FA" Ref="OPTION6"  Part="1"
+AR Path="/6009603F/603D70FA" Ref="ALTPLUS?"  Part="1"
+F 0 "OPTION6" H 18333 5373 60  0000 C CNN
+F 1 "MX-NoLED" H 18333 5299 20  0000 C CNN
+F 2 "MX_Only:MXOnly-1U-NoLEDHotswap" H 17675 5125 60  0001 C CNN
+F 3 "" H 17675 5125 60  0001 C CNN
+	1    18300 5150
+	1    0    0    -1
+$EndComp
+Wire Wire Line
+	17750 5300 18250 5300
+Wire Wire Line
+	18450 5100 18450 5000
+Wire Wire Line
+	18450 5000 17950 5000
+$Comp
+L MX_Alps_Hybrid:MX-NoLED OPTION2
+U 1 1 603FDE96
+P 17300 3600
+AR Path="/603FDE96" Ref="OPTION2"  Part="1"
+AR Path="/6009603F/603FDE96" Ref="ALTPLUS?"  Part="1"
+F 0 "OPTION2" H 17333 3823 60  0000 C CNN
+F 1 "MX-NoLED" H 17333 3749 20  0000 C CNN
+F 2 "MX_Only:MXOnly-1U-NoLEDHotswap" H 16675 3575 60  0001 C CNN
+F 3 "" H 16675 3575 60  0001 C CNN
+	1    17300 3600
+	1    0    0    -1
+$EndComp
+Wire Wire Line
+	16750 3750 17250 3750
+Wire Wire Line
+	17450 3550 17450 3450
+Wire Wire Line
+	17450 3450 16950 3450
 $EndSCHEMATC

Commit message: Rerouted
Parts:
- ALTENTER1, ALTPLUS1: footprint MX_Only:MXOnly-2U-ReversedStabilizers-NoLEDHotSwap -> MX_Only:MXOnly-2U-NoLEDHotswap
Connections:
- net COL0: now also ALTENTER1.1 (COL), ALTPLUS1.1 (COL), OPTION4.1 (COL); no longer ZERO2.1 (COL)
- net COL1: now also OPTION5.1 (COL), ZERO2.1 (COL); no longer OPTION4.1 (COL)
- net COL2: now also ALTZERO1.1 (COL)
- net COL3: now also OPTION2.1 (COL); no longer ALTENTER1.1 (COL), ALTPLUS1.1 (COL), ALTZERO1.1 (COL), OPTION5.1 (COL)
- net at D73.2 (A), SEVEN2.2 (ROW): now also ALTPLUS1.2 (ROW)
- net at D80.2 (A), ONE2.2 (ROW): now also ALTENTER1.2 (ROW)
- net at D83.2 (A): now also OPTION4.2 (ROW); no longer ZERO2.2 (ROW)
- net at D84.2 (A), DEL2.2 (ROW): now also ALTZERO1.2 (ROW)
- net at D85.2 (A), ENTER2.2 (ROW), OPTION6.2 (ROW): no longer ALTZERO1.2 (ROW), OPTION5.2 (ROW)
- net at D86.2 (A), OPTION1.2 (ROW): no longer ALTPLUS1.2 (ROW)
- net at D87.2 (A), OPTION3.2 (ROW): no longer ALTENTER1.2 (ROW)
- net at D88.2 (A): now also OPTION5.2 (ROW), ZERO2.2 (ROW); no longer OPTION4.2 (ROW)
Other:
- moved on the sheet: ALTZERO1, OPTION4, OPTION6, ZERO2
Changed lines of the file:
@@
 	1    0    0    -1
 $EndComp
-Wire Wire Line
-	15200 4550 15050 4550
 $Comp
 L Diode:1N4148 D80
@@
 L MX_Alps_Hybrid:MX-NoLED ZERO2
 U 1 1 6013051C
-P 15250 5150
+P 15800 5150
 AR Path="/6013051C" Ref="ZERO2"  Part="1"
 AR Path="/6009603F/6013051C" Ref="ZERO?"  Part="1"
-F 0 "ZERO2" H 15283 5373 60  0000 C CNN
-F 1 "MX-NoLED" H 15283 5299 20  0000 C CNN
-F 2 "MX_Only:MXOnly-2U-ReversedStabilizers-NoLEDHotSwap" H 14625 5125 60  0001 C CNN
-F 3 "" H 14625 5125 60  0001 C CNN
-	1    15250 5150
+F 0 "ZERO2" H 15833 5373 60  0000 C CNN
+F 1 "MX-NoLED" H 15833 5299 20  0000 C CNN
+F 2 "MX_Only:MXOnly-2U-ReversedStabilizers-NoLEDHotSwap" H 15175 5125 60  0001 C CNN
+F 3 "" H 15175 5125 60  0001 C CNN
+	1    15800 5150
 	1    0    0    -1
 $EndComp
@@
 $EndComp
 Wire Wire Line
-	16250 5300 16100 5300
+	16250 5300 16150 5300
 $Comp
 L Diode:1N4148 D84
@@
 Connection ~ 15400 2800
 Wire Wire Line
-	15400 2800 15400 2050
+	15400 2800 15400 2700
 Connection ~ 15400 3550
 Wire Wire Line
@@
 Connection ~ 15400 4350
 Wire Wire Line
-	15400 4350 15400 3550
-Wire Wire Line
 	15950 1800 15950 2050
 Connection ~ 15950 2050
@@
 	16950 1800 16950 2050
 Connection ~ 16950 2050
-Connection ~ 16950 3550
 Text GLabel 14850 2550 0    50   Input ~ 0
 ROW0
@@
 $EndComp
 Wire Wire Line
-	15750 5300 15600 5300
+	15750 5300 15650 5300
 $Comp
 L Diode:1N4148 D88
@@
 L MX_Alps_Hybrid:MX-NoLED OPTION4
 U 1 1 6019024A
-P 15800 5150
+P 15250 5150
 AR Path="/6019024A" Ref="OPTION4"  Part="1"
 AR Path="/6009603F/6019024A" Ref="OPTION?"  Part="1"
-F 0 "OPTION4" H 15833 5373 60  0000 C CNN
-F 1 "MX-NoLED" H 15833 5299 20  0000 C CNN
-F 2 "MX_Only:MXOnly-1U-NoLEDHotswap" H 15175 5125 60  0001 C CNN
-F 3 "" H 15175 5125 60  0001 C CNN
-	1    15800 5150
-	1    0    0    -1
-$EndComp
-Wire Wire Line
-	15950 4350 15950 5100
+F 0 "OPTION4" H 15283 5373 60  0000 C CNN
+F 1 "MX-NoLED" H 15283 5299 20  0000 C CNN
+F 2 "MX_Only:MXOnly-1U-NoLEDHotswap" H 14625 5125 60  0001 C CNN
+F 3 "" H 14625 5125 60  0001 C CNN
+	1    15250 5150
+	1    0    0    -1
+$EndComp
 Connection ~ 15950 4350
 Wire Wire Line
@@
 Connection ~ 16100 3300
 Connection ~ 16950 2800
-Connection ~ 16950 4350
 Connection ~ 15600 5600
 Wire Wire Line
@@
 	15600 5600 16100 5600
 Wire Wire Line
-	16950 3550 16950 4250
-Wire Wire Line
-	16950 4350 16950 5000
-Wire Wire Line
-	16950 2800 16950 3550
+	16950 2800 16950 3450
 $Comp
 L MX_Alps_Hybrid:MX-NoLED ALTPLUS1
@@
 F 0 "ALTPLUS1" H 17333 3073 60  0000 C CNN
 F 1 "MX-NoLED" H 17333 2999 20  0000 C CNN
-F 2 "MX_Only:MXOnly-2U-ReversedStabilizers-NoLEDHotSwap" H 16675 2825 60  0001 C CNN
+F 2 "MX_Only:MXOnly-2U-NoLEDHotswap" H 16675 2825 60  0001 C CNN
 F 3 "" H 16675 2825 60  0001 C CNN
 	1    17300 2850
@@
 $EndComp
 Wire Wire Line
-	16950 2050 16950 2700
-Wire Wire Line
-	16750 3000 17250 3000
-Connection ~ 16750 3000
-Wire Wire Line
 	17450 2800 17450 2700
-Wire Wire Line
-	17450 2700 16950 2700
-Connection ~ 16950 2700
-Wire Wire Line
-	16950 2700 16950 2800
 $Comp
 L MX_Alps_Hybrid:MX-NoLED ALTZERO1
 U 1 1 6031C7B4
-P 17300 5150
+P 16300 5800
 AR Path="/6031C7B4" Ref="ALTZERO1"  Part="1"
 AR Path="/6009603F/6031C7B4" Ref="ALTPLUS?"  Part="1"
-F 0 "ALTZERO1" H 17333 5373 60  0000 C CNN
-F 1 "MX-NoLED" H 17333 5299 20  0000 C CNN
-F 2 "MX_Only:MXOnly-2U-ReversedStabilizers-NoLEDHotSwap" H 16675 5125 60  0001 C CNN
-F 3 "" H 16675 5125 60  0001 C CNN
-	1    17300 5150
-	1    0    0    -1
-$EndComp
-Wire Wire Line
-	16750 5300 17250 5300
-Wire Wire Line
-	17450 5100 17450 5000
-Wire Wire Line
-	17450 5000 16950 5000
-Connection ~ 16950 5000
-Wire Wire Line
-	16950 5000 16950 5100
-Connection ~ 16750 5300
-$Comp
-L MX_Alps_Hybrid:MX-NoLED ALTENTER1
-U 1 1 6034204C
-P 17300 4400
-AR Path="/6034204C" Ref="ALTENTER1"  Part="1"
-AR Path="/6009603F/6034204C" Ref="ALTPLUS?"  Part="1"
-F 0 "ALTENTER1" H 17333 4623 60  0000 C CNN
-F 1 "MX-NoLED" H 17333 4549 20  0000 C CNN
-F 2 "MX_Only:MXOnly-2U-ReversedStabilizers-NoLEDHotSwap" H 16675 4375 60  0001 C CNN
-F 3 "" H 16675 4375 60  0001 C CNN
-	1    17300 4400
-	1    0    0    -1
-$EndComp
-Wire Wire Line
-	16750 4550 17250 4550
-Wire Wire Line
-	17450 4350 17450 4250
-Wire Wire Line
-	17450 4250 16950 4250
-Connection ~ 16950 4250
-Wire Wire Line
-	16950 4250 16950 4350
-Connection ~ 16750 4550
-$Comp
-L MX_Alps_Hybrid:MX-NoLED OPTION5
-U 1 1 603B6F36
-P 17800 5150
-AR Path="/603B6F36" Ref="OPTION5"  Part="1"
-AR Path="/6009603F/603B6F36" Ref="ALTPLUS?"  Part="1"
-F 0 "OPTION5" H 17833 5373 60  0000 C CNN
-F 1 "MX-NoLED" H 17833 5299 20  0000 C CNN
-F 2 "MX_Only:MXOnly-1U-NoLEDHotswap" H 17175 5125 60  0001 C CNN
-F 3 "" H 17175 5125 60  0001 C CNN
-	1    17800 5150
-	1    0    0    -1
-$EndComp
-Wire Wire Line
-	17250 5300 17750 5300
-Wire Wire Line
-	17950 5100 17950 5000
-Wire Wire Line
-	17950 5000 17450 5000
-$Comp
-L MX_Alps_Hybrid:MX-NoLED OPTION6
-U 1 1 603D70FA
-P 18300 5150
-AR Path="/603D70FA" Ref="OPTION6"  Part="1"
-AR Path="/6009603F/603D70FA" Ref="ALTPLUS?"  Part="1"
-F 0 "OPTION6" H 18333 5373 60  0000 C CNN
-F 1 "MX-NoLED" H 18333 5299 20  0000 C CNN
-F 2 "MX_Only:MXOnly-1U-NoLEDHotswap" H 17675 5125 60  0001 C CNN
-F 3 "" H 17675 5125 60  0001 C CNN
-	1    18300 5150
-	1    0    0    -1
-$EndComp
-Wire Wire Line
-	17750 5300 18250 5300
-Wire Wire Line
-	18450 5100 18450 5000
-Wire Wire Line
-	18450 5000 17950 5000
+F 0 "ALTZERO1" H 16333 6023 60  0000 C CNN
+F 1 "MX-NoLED" H 16333 5949 20  0000 C CNN
+F 2 "MX_Only:MXOnly-2U-ReversedStabilizers-NoLEDHotSwap" H 15675 5775 60  0001 C CNN
+F 3 "" H 15675 5775 60  0001 C CNN
+	1    16300 5800
+	1    0    0    -1
+$EndComp
 $Comp
 L MX_Alps_Hybrid:MX-NoLED OPTION2
@@
 Wire Wire Line
 	17450 3450 16950 3450
+Wire Wire Line
+	16950 2050 16950 2700
+Wire Wire Line
+	16950 2700 16950 2800
+Connection ~ 15400 2700
+Wire Wire Line
+	15400 2700 15400 2050
+Wire Wire Line
+	15400 2700 17450 2700
+Wire Wire Line
+	15950 4350 15950 5100
+$Comp
+L MX_Alps_Hybrid:MX-NoLED OPTION5
+U 1 1 6067C027
+P 15800 5800
+AR Path="/6067C027" Ref="OPTION5"  Part="1"
+AR Path="/6009603F/6067C027" Ref="OPTION?"  Part="1"
+F 0 "OPTION5" H 15833 6023 60  0000 C CNN
+F 1 "MX-NoLED" H 15833 5949 20  0000 C CNN
+F 2 "MX_Only:MXOnly-1U-NoLEDHotswap" H 15175 5775 60  0001 C CNN
+F 3 "" H 15175 5775 60  0001 C CNN
+	1    15800 5800
+	1    0    0    -1
+$EndComp
+Wire Wire Line
+	15750 5950 15650 5950
+Wire Wire Line
+	15650 5950 15650 5300
+Connection ~ 15650 5300
+Wire Wire Line
+	15650 5300 15600 5300
+Wire Wire Line
+	15950 5750 15950 5100
+Connection ~ 15950 5100
+Connection ~ 16950 3450
+Wire Wire Line
+	16950 3450 16950 3550
+Wire Wire Line
+	16950 4350 16950 5000
+Wire Wire Line
+	17450 5100 17450 5000
+$Comp
+L MX_Alps_Hybrid:MX-NoLED OPTION6
+U 1 1 603D70FA
+P 17300 5150
+AR Path="/603D70FA" Ref="OPTION6"  Part="1"
+AR Path="/6009603F/603D70FA" Ref="ALTPLUS?"  Part="1"
+F 0 "OPTION6" H 17333 5373 60  0000 C CNN
+F 1 "MX-NoLED" H 17333 5299 20  0000 C CNN
+F 2 "MX_Only:MXOnly-1U-NoLEDHotswap" H 16675 5125 60  0001 C CNN
+F 3 "" H 16675 5125 60  0001 C CNN
+	1    17300 5150
+	1    0    0    -1
+$EndComp
+Wire Wire Line
+	16750 5300 17250 5300
+Connection ~ 16750 5300
+Wire Wire Line
+	17450 5000 16950 5000
+Connection ~ 16950 5000
+Wire Wire Line
+	16950 5000 16950 5100
+Wire Wire Line
+	16450 5100 16450 5750
+Connection ~ 16450 5100
+Wire Wire Line
+	16250 5950 16150 5950
+Wire Wire Line
+	16150 5950 16150 5300
+Connection ~ 16150 5300
+Wire Wire Line
+	16150 5300 16100 5300
+Connection ~ 16950 4350
+Connection ~ 16950 3550
+Wire Wire Line
+	15200 4550 15050 4550
+Wire Wire Line
+	16950 4250 16950 3550
+Wire Wire Line
+	16950 4350 16950 4250
+Wire Wire Line
+	17450 4350 17450 4250
+Wire Wire Line
+	15400 4250 15400 3550
+Wire Wire Line
+	15400 4350 15400 4250
+Connection ~ 15400 4250
+Wire Wire Line
+	15400 4250 17450 4250
+$Comp
+L MX_Alps_Hybrid:MX-NoLED ALTENTER1
+U 1 1 6034204C
+P 17300 4400
+AR Path="/6034204C" Ref="ALTENTER1"  Part="1"
+AR Path="/6009603F/6034204C" Ref="ALTPLUS?"  Part="1"
+F 0 "ALTENTER1" H 17333 4623 60  0000 C CNN
+F 1 "MX-NoLED" H 17333 4549 20  0000 C CNN
+F 2 "MX_Only:MXOnly-2U-NoLEDHotswap" H 16675 4375 60  0001 C CNN
+F 3 "" H 16675 4375 60  0001 C CNN
+	1    17300 4400
+	1    0    0    -1
+$EndComp
+Wire Wire Line
+	17050 4550 17050 4500
+Wire Wire Line
+	17050 4500 15300 4500
+Wire Wire Line
+	15300 4500 15300 4550
+Wire Wire Line
+	15300 4550 15200 4550
+Wire Wire Line
+	17050 4550 17250 4550
+Connection ~ 15200 4550
+Wire Wire Line
+	17250 3000 17050 3000
+Wire Wire Line
+	17050 3000 17050 2950
+Wire Wire Line
+	17050 2950 15300 2950
+Wire Wire Line
+	15300 2950 15300 3000
+Wire Wire Line
+	15300 3000 15200 3000
+Connection ~ 15200 3000
 $EndSCHEMATC
