File: 65NumpadBACKUP.kicad_pcb (KiCad board)
At the start: 2 copper layers, 423.9 x 98.4 mm, 193 parts, among them J1 MX-NoLED, K1 MX-NoLED, M1 MX-NoLED, P1 MX-NoLED, Q1 MX-NoLED, T1 MX-NoLED, U2 MX-NoLED, X1 MX-NoLED, Y1 MX-NoLED

Commit message: Removed traces
Parts:
- removed the DEL2 at (338.9, 134.9)
- removed the DEL2 at (396.1, 134.9)
- removed the DEL2 at (377.0, 134.9)
- removed the FOUR2 at (396.1, 96.8)
- removed the ONE2 at (396.1, 115.9)
- removed the REF** at (401.6, 35.7)
- removed the REF** at (430.2, 154.8)
- removed the REF** at (333.4, 33.3)
- removed the REF** at (335.0, 159.5)
- removed the SEVEN2 at (396.1, 77.8)
- added REF**: MountingHole_3.2mm_M3, Mounting_Holes:MountingHole_3.2mm_M3, B.Cu at (403.2, 51.6)
- added REF**: MountingHole_3.2mm_M3, Mounting_Holes:MountingHole_3.2mm_M3, B.Cu at (403.2, 106.4)
- added REF**: MountingHole_3.2mm_M3, Mounting_Holes:MountingHole_3.2mm_M3, B.Cu at (331.8, 71.4)
- added REF**: MountingHole_3.2mm_M3, Mounting_Holes:MountingHole_3.2mm_M3, B.Cu at (348.5, 125.4)
- POGO1, POGO3: footprint 65Numpad:PogoConnector -> Pin_Headers:Pin_Header_Angled_1x04_Pitch2.54mm
- POGO2, POGO4: footprint 65Numpad:PogoConnectorMirrored -> Pin_Headers:Pin_Header_Angled_1x04_Pitch2.54mm
- moved DEL2 19.1 mm to (377.0, 134.9)
- moved Numpad1 19.1 mm to (358.0, 65.9)
- moved ZERO2 19.1 mm to (386.6, 154.0)
- moved PLUS1 19.0 mm to (319.9, 125.4)
- moved PLUS1 19.0 mm to (319.9, 87.3)
Routing:
- net COL3: track 0.00 -> 590.2 mm, vias 0 -> 22
- net COL2: track 0.00 -> 540.7 mm, vias 0 -> 10
- net SERIAL: track 0.00 -> 504.2 mm, vias 0 -> 7
- net COL4: track 0.00 -> 504.2 mm, vias 0 -> 17
- net GND: track 0.00 -> 489.8 mm, vias 0 -> 10
- net VCC: track 0.00 -> 488.8 mm, vias 0 -> 12
- net COL6: track 0.00 -> 454.2 mm, vias 0 -> 12
- net COL5: track 0.00 -> 449.8 mm, vias 0 -> 14
- net ROW4: track 0.00 -> 430.6 mm, vias 0 -> 1
- net COL1: track 0.00 -> 418.5 mm, vias 0 -> 12
- net COL0: track 0.00 -> 397.6 mm, vias 0 -> 7
- net ROW3: track 0.00 -> 375.1 mm, vias 0 -> 13
- net ROW2: track 0.00 -> 372.2 mm, vias 0 -> 2
- net ROW8: track 0.00 -> 365.3 mm
- net ROW1: track 0.00 -> 357.4 mm, vias 0 -> 12
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
Commit message: Created FR4 plate
Parts:
- removed ESC1: MX-NoLED, MX_Only:MXOnly-1U-NoLEDHotswap
- removed the PLUS1 at (319.9, 125.4)
- removed the PLUS1 at (319.9, 87.3)
- removed the REF** at (403.2, 51.6)
- removed the REF** at (148.4, 68.6)
- removed the REF** at (403.2, 106.4)
- removed the REF** at (331.8, 71.4)
- removed the REF** at (348.5, 125.4)
- removed the REF** at (280.2, 59.5)
- removed the REF** at (238.9, 134.9)
- removed the REF** at (-0.79, 77.8)
- removed the REF** at (153.2, 134.9)
- removed the REF** at (45.2, 134.9)
- removed the ZERO2 at (386.6, 154.0)
- added ALTENTER1: MX-NoLED, MX_Only:MXOnly-2U-ReversedStabilizers-NoLEDHotSwap, F.Cu at (338.9, 125.4)
- added ALTPLUS1: MX-NoLED, MX_Only:MXOnly-2U-ReversedStabilizers-NoLEDHotSwap, F.Cu at (338.9, 87.3)
- added ALTZERO1: MX-NoLED, MX_Only:MXOnly-2U-ReversedStabilizers-NoLEDHotSwap, F.Cu at (386.6, 134.9)
- added D86: 1N4148, 65Numpad:D_DO-35_SOD27_P7.62mm_HorizontalMovedText, B.Cu at (381.0, 85.7)
- added D87: 1N4148, 65Numpad:D_DO-35_SOD27_P7.62mm_HorizontalMovedText, B.Cu at (400.1, 104.8)
- added D88: 1N4148, 65Numpad:D_DO-35_SOD27_P7.62mm_HorizontalMovedText, B.Cu at (371.5, 131.0)
- added ESC: MX-NoLED, MX_Only:MXOnly-1U-NoLEDHotswap, F.Cu at (5.56, 58.7)
- added OPTION1: MX-NoLED, MX_Only:MXOnly-1U-NoLEDHotswap, F.Cu at (396.1, 77.8)
- added OPTION2: MX-NoLED, MX_Only:MXOnly-1U-NoLEDHotswap, F.Cu at (396.1, 96.8)
- added OPTION3: MX-NoLED, MX_Only:MXOnly-1U-NoLEDHotswap, F.Cu at (396.1, 115.9)
- added OPTION4: MX-NoLED, MX_Only:MXOnly-1U-NoLEDHotswap, F.Cu at (338.9, 134.9)
- added OPTION5: MX-NoLED, MX_Only:MXOnly-1U-NoLEDHotswap, F.Cu at (358.0, 134.9)
- added OPTION6: MX-NoLED, MX_Only:MXOnly-1U-NoLEDHotswap, F.Cu at (396.1, 134.9)
- added REF**: MountingHole_4.22mm_M2INSERT, 65Numpad:MountingHole_4.22mm_M2INSERT, B.Cu at (23.0, 77.8)
- added REF**: MountingHole_4.22mm_M2INSERT, 65Numpad:MountingHole_4.22mm_M2INSERT, B.Cu at (86.5, 125.4)
- added REF**: MountingHole_4.22mm_M2INSERT, 65Numpad:MountingHole_4.22mm_M2INSERT, B.Cu at (281.8, 87.3)
- added REF**: MountingHole_4.22mm_M2INSERT, 65Numpad:MountingHole_4.22mm_M2INSERT, B.Cu at (91.3, 68.3)
- added REF**: MountingHole_4.22mm_M2INSERT, 65Numpad:MountingHole_4.22mm_M2INSERT, B.Cu at (210.3, 125.4)
- added REF**: MountingHole_4.22mm_M2INSERT, 65Numpad:MountingHole_4.22mm_M2INSERT, B.Cu at (205.6, 68.3)
- added REF**: MountingHole_4.22mm_M2INSERT, 65Numpad:MountingHole_4.22mm_M2INSERT, B.Cu at (331.2, 68.3)
- added REF**: MountingHole_4.22mm_M2INSERT, 65Numpad:MountingHole_4.22mm_M2INSERT, B.Cu at (403.6, 68.3)
- added REF**: MountingHole_4.22mm_M2INSERT, 65Numpad:MountingHole_4.22mm_M2INSERT, B.Cu at (367.5, 125.4)
- D1, D10, D11, D12, D13, D14, D15, D16, D17, D18, D19, D2, D20, D21, D22, D23, D24, D25, D26, D27, D28, D3, D30, D31, D32, D33, D34, D35, D36, D37, D38, D39, D4, D40, D41, D42, D43, D44, D45, D46, D47, D48, D49, D5, D50, D51, D52, D53, D54, D55, D56, D57, D58, D59, D6, D60, D61, D62, D63, D64, D65, D66, D67, D68, D69, D7, D70, D71, D72, D73, D74, D75, D76, D77, D78, D79, D8, D80, D81, D82, D83, D84, D85, D9: footprint Diodes_THT:D_DO-35_SOD27_P7.62mm_Horizontal -> 65Numpad:D_DO-35_SOD27_P7.62mm_HorizontalMovedText
- ENTER2, PLUS1, ZERO2: footprint MX_Only:MXOnly-2U-NoLEDHotswap -> MX_Only:MXOnly-2U-ReversedStabilizers-NoLEDHotSwap
- POGO1, POGO3: footprint Pin_Headers:Pin_Header_Angled_1x04_Pitch2.54mm -> 65Numpad:PogoConnector
- POGO2, POGO4: footprint Pin_Headers:Pin_Header_Angled_1x04_Pitch2.54mm -> 65Numpad:PogoConnectorMirrored
- SPACE1: footprint MX_Only:MXOnly-6.25U-NoLEDHotswap -> MX_Only:MXOnly-6.25U-ReversedStabilizers-NoLEDHotswap
- moved D85 21.7 mm to (381.0, 123.0)
- moved D73 19.3 mm to (361.9, 82.5)
- moved D30 19.2 mm to (20.6, 102.1)
- moved D80 19.1 mm to (361.9, 123.0)
- moved D83 19.1 mm to (371.5, 142.1)
- moved D70 19.1 mm to (381.0, 66.7)
- moved D64 15.9 mm to (245.3, 140.5)
- moved D84 10.3 mm to (371.5, 138.9)
- moved D79 6.35 mm to (400.1, 101.6)
- moved D81 3.97 mm to (361.9, 119.9)
- moved D82 3.97 mm to (381.0, 119.9)
- moved D71 3.17 mm to (381.0, 63.5)
- moved D75 3.17 mm to (381.0, 82.5)
- moved D69 1.59 mm to (342.9, 65.1)
- moved D72 1.59 mm to (400.1, 65.1)
- renumbered FIVE1 to FIVE, FOUR1 to FOUR, ONE1 to ONE, SIX1 to SIX, THREE1 to THREE, TWO1 to TWO
Connections:
- ZERO2 pad 1: COL0 -> COL1
- ZERO2 pad 2: Net-(D83-Pad2) -> Net-(D88-Pad2)
Routing:
- net COL0: track 397.6 -> 299.2 mm, vias 7 -> 0
- net COL3: track 590.2 -> 515.4 mm, vias 22 -> 3
- net COL2: track 540.7 -> 469.7 mm, vias 10 -> 7
- net ROW4: track 430.6 -> 368.7 mm, vias 1 -> 4
- net COL4: track 504.2 -> 452.9 mm, vias 17 -> 2
- net COL5: track 449.8 -> 400.0 mm, vias 14 -> 2
- net COL1: track 418.5 -> 369.1 mm, vias 12 -> 2
- net GND: track 489.8 -> 441.0 mm, vias 10 -> 2
- net COL6: track 454.2 -> 414.0 mm, vias 12 -> 1
- net SERIAL: track 504.2 -> 468.3 mm, vias 7 -> 0
- net Net-(D86-Pad2): track 0.00 -> 31.7 mm
- net Net-(D85-Pad2): track 16.1 -> 43.4 mm
- net ROW6: track 321.4 -> 294.6 mm
- net ROW1: track 357.4 -> 331.2 mm, vias 12 -> 1
- net Net-(CAPS1-Pad2): track 32.7 -> 6.52 mm
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