File: 65Numpad.kicad_pcb (KiCad board)
At the start: 2 copper layers, 412.8 x 98.4 mm, 174 parts, among them J1 MX-NoLED, K1 MX-NoLED, M1 MX-NoLED, P1 MX-NoLED, Q1 MX-NoLED, T1 MX-NoLED, U2 MX-NoLED, X1 MX-NoLED, Y1 MX-NoLED

Commit message: Removed traces
Parts:
- added DEL2: MX-NoLED, MX_Only:MXOnly-1U-NoLEDHotswap, F.Cu at (338.9, 134.9)
- added DEL2: MX-NoLED, MX_Only:MXOnly-1U-NoLEDHotswap, F.Cu at (396.1, 134.9)
- added DEL2: MX-NoLED, MX_Only:MXOnly-1U-NoLEDHotswap, F.Cu at (377.0, 134.9)
- added FOUR2: MX-NoLED, MX_Only:MXOnly-1U-NoLEDHotswap, F.Cu at (396.1, 96.8)
- added ONE2: MX-NoLED, MX_Only:MXOnly-1U-NoLEDHotswap, F.Cu at (396.1, 115.9)
- added PLUS1: MX-NoLED, MX_Only:MXOnly-2U-NoLEDHotswap, F.Cu at (338.9, 125.4)
- added PLUS1: MX-NoLED, MX_Only:MXOnly-2U-NoLEDHotswap, F.Cu at (338.9, 87.3)
- added REF**: MountingHole_3.2mm_M3, Mounting_Holes:MountingHole_3.2mm_M3, B.Cu at (401.6, 35.7)
- added REF**: MountingHole_3.2mm_M3, Mounting_Holes:MountingHole_3.2mm_M3, B.Cu at (148.4, 68.6)
- added REF**: MountingHole_3.2mm_M3, Mounting_Holes:MountingHole_3.2mm_M3, B.Cu at (430.2, 154.8)
- added REF**: MountingHole_3.2mm_M3, Mounting_Holes:MountingHole_3.2mm_M3, B.Cu at (333.4, 33.3)
- added REF**: MountingHole_3.2mm_M3, Mounting_Holes:MountingHole_3.2mm_M3, B.Cu at (335.0, 159.5)
- added REF**: MountingHole_3.2mm_M3, Mounting_Holes:MountingHole_3.2mm_M3, B.Cu at (280.2, 59.5)
- added REF**: MountingHole_3.2mm_M3, Mounting_Holes:MountingHole_3.2mm_M3, B.Cu at (238.9, 134.9)
- added REF**: MountingHole_3.2mm_M3, Mounting_Holes:MountingHole_3.2mm_M3, B.Cu at (-0.79, 77.8)
- added REF**: MountingHole_3.2mm_M3, Mounting_Holes:MountingHole_3.2mm_M3, B.Cu at (153.2, 134.9)
- added REF**: MountingHole_3.2mm_M3, Mounting_Holes:MountingHole_3.2mm_M3, B.Cu at (45.2, 134.9)
- added SEVEN2: MX-NoLED, MX_Only:MXOnly-1U-NoLEDHotswap, F.Cu at (396.1, 77.8)
- added ZERO2: MX-NoLED, MX_Only:MXOnly-2U-NoLEDHotswap, F.Cu at (386.6, 134.9)
- POGO1, POGO3: footprint Pin_Headers:Pin_Header_Angled_1x04_Pitch2.54mm -> 65Numpad:PogoConnector
- POGO2, POGO4: footprint Pin_Headers:Pin_Header_Angled_1x04_Pitch2.54mm -> 65Numpad:PogoConnectorMirrored
- moved D30 19.2 mm to (23.0, 83.0)
- moved DEL2 19.1 mm to (358.0, 134.9)
- moved Numpad1 19.1 mm to (377.0, 65.9)
- moved POGO2 7.14 mm to (305.6, 55.6)
- moved POGO3 7.14 mm to (324.6, 55.6)
- moved POGO1 7.14 mm to (-8.73, 55.6)
- moved POGO4 7.14 mm to (410.4, 55.6)
Routing:
- net COL3: track 590.2 -> 0.00 mm, vias 22 -> 0
- net COL2: track 539.5 -> 0.00 mm, vias 10 -> 0
- net COL4: track 504.2 -> 0.00 mm, vias 17 -> 0
- net SERIAL: track 491.4 -> 0.00 mm, vias 7 -> 0
- net VCC: track 459.7 -> 0.00 mm, vias 12 -> 0
- net GND: track 458.8 -> 0.00 mm, vias 10 -> 0
- net COL6: track 453.7 -> 0.00 mm, vias 12 -> 0
- net COL5: track 449.8 -> 0.00 mm, vias 14 -> 0
- net COL1: track 418.5 -> 0.00 mm, vias 12 -> 0
- net ROW4: track 417.9 -> 0.00 mm
- net COL0: track 397.6 -> 0.00 mm, vias 7 -> 0
- net ROW3: track 373.1 -> 0.00 mm, vias 13 -> 0
- net ROW2: track 372.2 -> 0.00 mm, vias 2 -> 0
- net ROW8: track 365.3 -> 0.00 mm
- net ROW1: track 357.6 -> 0.00 mm, vias 12 -> 0
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Other:
- board size 412.8 x 98.4 mm -> 423.9 x 98.4 mm

Commit message: Schematic 1u addons
Parts:
- removed the DEL2 at (338.9, 134.9)
- removed the DEL2 at (396.1, 134.9)
- removed the DEL2 at (358.0, 134.9)
- removed the FOUR2 at (396.1, 96.8)
- removed the ONE2 at (396.1, 115.9)
- removed the PLUS1 at (338.9, 125.4)
- removed the PLUS1 at (338.9, 87.3)
- removed the SEVEN2 at (396.1, 77.8)
- removed the ZERO2 at (386.6, 134.9)
- added ALTENTER1: MX-NoLED, MX_Only:MXOnly-2U-ReversedStabilizers-NoLEDHotSwap, F.Cu at (338.9, 125.4)
- added ALTPLUS1: MX-NoLED, MX_Only:MXOnly-2U-ReversedStabilizers-NoLEDHotSwap, F.Cu at (338.9, 87.3)
- added ALTZERO1: MX-NoLED, MX_Only:MXOnly-2U-ReversedStabilizers-NoLEDHotSwap, F.Cu at (386.6, 134.9)
- added D86: 1N4148, Diodes_THT:D_DO-35_SOD27_P7.62mm_Horizontal, B.Cu at (373.4, 85.7)
- added D87: 1N4148, Diodes_THT:D_DO-35_SOD27_P7.62mm_Horizontal, B.Cu at (342.9, 107.2)
- added D88: 1N4148, Diodes_THT:D_DO-35_SOD27_P7.62mm_Horizontal, B.Cu at (365.9, 124.3)
- added OPTION1: MX-NoLED, MX_Only:MXOnly-1U-NoLEDHotswap, F.Cu at (396.1, 77.8)
- added OPTION2: MX-NoLED, MX_Only:MXOnly-1U-NoLEDHotswap, F.Cu at (396.1, 96.8)
- added OPTION3: MX-NoLED, MX_Only:MXOnly-1U-NoLEDHotswap, F.Cu at (396.1, 115.9)
- added OPTION4: MX-NoLED, MX_Only:MXOnly-1U-NoLEDHotswap, F.Cu at (338.9, 134.9)
- added OPTION5: MX-NoLED, MX_Only:MXOnly-1U-NoLEDHotswap, F.Cu at (358.0, 134.9)
- added OPTION6: MX-NoLED, MX_Only:MXOnly-1U-NoLEDHotswap, F.Cu at (396.1, 134.9)
- ENTER2, PLUS1, ZERO2: footprint MX_Only:MXOnly-2U-NoLEDHotswap -> MX_Only:MXOnly-2U-ReversedStabilizers-NoLEDHotSwap
- SPACE1: footprint MX_Only:MXOnly-6.25U-NoLEDHotswap -> MX_Only:MXOnly-6.25U-ReversedStabilizers-NoLEDHotswap
- moved D85 21.7 mm to (381.0, 123.0)
- moved D80 19.5 mm to (361.9, 119.9)
- moved D83 19.5 mm to (371.5, 138.9)
- moved D73 19.3 mm to (361.9, 82.5)
- moved Numpad1 19.1 mm to (358.0, 65.9)
- moved REF** 12.1 mm to (332.6, 171.4)
- moved D84 9.56 mm to (371.5, 142.1)
- moved D79 9.53 mm to (400.1, 104.8)
- moved D82 3.97 mm to (381.0, 119.9)
- moved D75 3.17 mm to (381.0, 82.5)
- moved D81 0.79 mm to (361.9, 123.0)
Connections:
- DEL2 pad 1: (no net) -> COL2
- DEL2 pad 2: (no net) -> Net-(D84-Pad2)

Commit message: Rerouted
Parts:
- removed the REF** at (401.6, 35.7)
- removed the REF** at (430.2, 154.8)
- removed the REF** at (333.4, 33.3)
- added REF**: MountingHole_3.2mm_M3, Mounting_Holes:MountingHole_3.2mm_M3, B.Cu at (67.5, 125.4)
- added REF**: MountingHole_3.2mm_M3, Mounting_Holes:MountingHole_3.2mm_M3, B.Cu at (62.7, 68.3)
- added REF**: MountingHole_3.2mm_M3, Mounting_Holes:MountingHole_3.2mm_M3, B.Cu at (403.6, 70.4)
- added REF**: MountingHole_3.2mm_M3, Mounting_Holes:MountingHole_3.2mm_M3, B.Cu at (384.2, 142.1)
- added REF**: MountingHole_3.2mm_M3, Mounting_Holes:MountingHole_3.2mm_M3, B.Cu at (331.2, 69.8)
- ALTENTER1, ALTPLUS1: footprint MX_Only:MXOnly-2U-ReversedStabilizers-NoLEDHotSwap -> MX_Only:MXOnly-2U-NoLEDHotswap
- moved D87 57.2 mm to (400.1, 104.8)
- moved REF** 33.4 mm to (348.5, 142.1)
- moved D30 19.2 mm to (20.6, 102.1)
- moved D86 7.62 mm to (381.0, 85.7), turned to 180 degrees
- moved D79 3.18 mm to (400.1, 101.6)
- moved D83 3.18 mm to (371.5, 142.1)
- moved D84 3.18 mm to (371.5, 138.9)
- moved D80 3.17 mm to (361.9, 123.0)
- moved D81 3.17 mm to (361.9, 119.9)
Connections:
- ALTENTER1 pad 1: COL3 -> COL0
- ALTPLUS1 pad 1: COL3 -> COL0
- ALTZERO1 pad 1: COL3 -> COL2
- D73 pad 2: Net-(D73-Pad2) -> Net-(ALTPLUS1-Pad2)
- D80 pad 2: Net-(D80-Pad2) -> Net-(ALTENTER1-Pad2)
- D84 pad 2: Net-(D84-Pad2) -> Net-(ALTZERO1-Pad2)
- D85 pad 2: Net-(ALTZERO1-Pad2) -> Net-(D85-Pad2)
- D86 pad 2: Net-(ALTPLUS1-Pad2) -> Net-(D86-Pad2)
- D87 pad 2: Net-(ALTENTER1-Pad2) -> Net-(D87-Pad2)
- DEL2 pad 2: Net-(D84-Pad2) -> Net-(ALTZERO1-Pad2)
- ENTER2 pad 2: Net-(ALTZERO1-Pad2) -> Net-(D85-Pad2)
- ONE2 pad 2: Net-(D80-Pad2) -> Net-(ALTENTER1-Pad2)
- OPTION1 pad 2: Net-(ALTPLUS1-Pad2) -> Net-(D86-Pad2)
- OPTION2 pad 1: (no net) -> COL3
- OPTION3 pad 2: Net-(ALTENTER1-Pad2) -> Net-(D87-Pad2)
- OPTION4 pad 1: COL1 -> COL0
- OPTION4 pad 2: Net-(D88-Pad2) -> Net-(D83-Pad2)
- OPTION5 pad 1: COL3 -> COL1
- OPTION5 pad 2: Net-(ALTZERO1-Pad2) -> Net-(D88-Pad2)
- OPTION6 pad 2: Net-(ALTZERO1-Pad2) -> Net-(D85-Pad2)
- SEVEN2 pad 2: Net-(D73-Pad2) -> Net-(ALTPLUS1-Pad2)
- ZERO2 pad 1: COL0 -> COL1
- ZERO2 pad 2: Net-(D83-Pad2) -> Net-(D88-Pad2)
Routing:
- net COL3: track 0.00 -> 510.6 mm, vias 0 -> 3
- net COL2: track 0.00 -> 470.4 mm, vias 0 -> 7
- net SERIAL: track 0.00 -> 468.3 mm
- net VCC: track 0.00 -> 466.1 mm, vias 0 -> 4
- net COL4: track 0.00 -> 452.9 mm, vias 0 -> 2
- net GND: track 0.00 -> 441.0 mm, vias 0 -> 2
- net COL6: track 0.00 -> 411.5 mm, vias 0 -> 1
- net COL5: track 0.00 -> 400.0 mm, vias 0 -> 2
- net ROW3: track 0.00 -> 372.4 mm, vias 0 -> 5
- net COL1: track 0.00 -> 369.1 mm, vias 0 -> 2
- net ROW2: track 0.00 -> 367.8 mm, vias 0 -> 3
- net ROW0: track 0.00 -> 356.5 mm, vias 0 -> 6
- net ROW8: track 0.00 -> 352.5 mm
- net ROW4: track 0.00 -> 317.6 mm, vias 0 -> 3
- net ROW5: track 0.00 -> 313.5 mm, vias 0 -> 2
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
Commit message: Double checking tracks
Parts:
- added REF**: MountingHole_3.2mm_M3, Mounting_Holes:MountingHole_3.2mm_M3, B.Cu at (234.2, 125.4)
- added REF**: MountingHole_3.2mm_M3, Mounting_Holes:MountingHole_3.2mm_M3, B.Cu at (234.2, 68.3)
- ALTENTER1, ALTPLUS1: footprint MX_Only:MXOnly-2U-NoLEDHotswap -> MX_Only:MXOnly-2U-ReversedStabilizers-NoLEDHotSwap
Routing:
- net ROW1: track 246.0 -> 328.9 mm, vias 0 -> 1
- net ROW6: track 241.3 -> 294.6 mm
- net ROW4: track 317.6 -> 368.7 mm, vias 3 -> 5
- net ROW7: track 284.9 -> 331.1 mm
- net ROW9: track 293.9 -> 339.0 mm
- net COL3: track 510.6 -> 524.7 mm
- net COL6: track 411.5 -> 414.0 mm
- net ROW0: track 356.5 -> 355.9 mm

Commit message: Silkscreen changes
Parts:
- removed ESC1: MX-NoLED, MX_Only:MXOnly-1U-NoLEDHotswap
- added ESC: MX-NoLED, MX_Only:MXOnly-1U-NoLEDHotswap, F.Cu at (5.56, 58.7)
- renumbered FOUR1 to FOUR, ONE1 to ONE, THREE1 to THREE, TWO1 to TWO

Commit message: Created FR4 plate
Parts:
- removed the REF** at (238.9, 134.9)
- removed the REF** at (-0.79, 77.8)
- removed the REF** at (153.2, 134.9)
- removed the REF** at (45.2, 134.9)
- removed the REF** at (148.4, 68.6)
- removed the REF** at (384.2, 142.1)
- removed the REF** at (348.5, 142.1)
- removed the REF** at (331.2, 69.8)
- removed the REF** at (234.2, 125.4)
- removed the REF** at (234.2, 68.3)
- removed the REF** at (62.7, 68.3)
- added REF**: MountingHole_4.22mm_M2INSERT, 65Numpad:MountingHole_4.22mm_M2INSERT, B.Cu at (23.0, 77.8)
- added REF**: MountingHole_4.22mm_M2INSERT, 65Numpad:MountingHole_4.22mm_M2INSERT, B.Cu at (91.3, 68.3)
- added REF**: MountingHole_4.22mm_M2INSERT, 65Numpad:MountingHole_4.22mm_M2INSERT, B.Cu at (210.3, 125.4)
- added REF**: MountingHole_4.22mm_M2INSERT, 65Numpad:MountingHole_4.22mm_M2INSERT, B.Cu at (205.6, 68.3)
- added REF**: MountingHole_4.22mm_M2INSERT, 65Numpad:MountingHole_4.22mm_M2INSERT, B.Cu at (331.2, 68.3)
- added REF**: MountingHole_4.22mm_M2INSERT, 65Numpad:MountingHole_4.22mm_M2INSERT, B.Cu at (367.5, 125.4)
- D1, D10, D11, D12, D13, D14, D15, D16, D17, D18, D19, D2, D20, D21, D22, D23, D24, D25, D26, D27, D28, D3, D30, D31, D32, D33, D34, D35, D36, D37, D38, D39, D4, D40, D41, D42, D43, D44, D45, D46, D47, D48, D49, D5, D50, D51, D52, D53, D54, D55, D56, D57, D58, D59, D6, D60, D61, D62, D63, D64, D65, D66, D67, D68, D69, D7, D70, D71, D72, D73, D74, D75, D76, D77, D78, D79, D8, D80, D81, D82, D83, D84, D85, D86, D87, D88, D9: footprint Diodes_THT:D_DO-35_SOD27_P7.62mm_Horizontal -> 65Numpad:D_DO-35_SOD27_P7.62mm_HorizontalMovedText
- REF** (x3): value MountingHole_3.2mm_M3 -> MountingHole_4.22mm_M2INSERT; footprint Mounting_Holes:MountingHole_3.2mm_M3 -> 65Numpad:MountingHole_4.22mm_M2INSERT
- moved REF** 27.8 mm to (281.8, 87.3)
- moved D70 19.1 mm to (381.0, 66.7)
- moved REF** 19.0 mm to (86.5, 125.4)
- moved D64 15.9 mm to (245.3, 140.5)
- moved D88 8.68 mm to (371.5, 131.0), turned to 180 degrees
- moved D71 3.17 mm to (381.0, 63.5)
- moved REF** 2.10 mm to (403.6, 68.3)
- moved D69 1.59 mm to (342.9, 65.1)
- moved D72 1.59 mm to (400.1, 65.1)
- renumbered FIVE1 to FIVE, SIX1 to SIX
Routing:
- net Net-(D88-Pad2): track 24.9 -> 13.3 mm
- net COL3: track 524.7 -> 515.4 mm
- net ROW0: track 355.9 -> 347.3 mm, vias 6 -> 4
- net Net-(D70-Pad2): track 15.6 -> 23.9 mm, vias 0 -> 2
- net Net-(D64-Pad2): track 6.52 -> 11.7 mm
- net ROW1: track 328.9 -> 331.2 mm
- net Net-(ASTERISK1-Pad2): track 15.6 -> 13.8 mm
- net ROW8: track 352.5 -> 351.2 mm
- net COL2: track 470.4 -> 469.7 mm
- net Net-(D72-Pad2): track 15.6 -> 14.9 mm
- net Net-(D69-Pad2): track 15.6 -> 14.9 mm
- net ROW7: track 331.1 -> 330.4 mm
- net ROW4: vias 5 -> 4
- net ROW3: vias 5 -> 4

Commit message: Forgot the solder mask :(
Parts:
- moved POGO1 5.56 mm to (-3.17, 55.6)
- moved POGO2 5.56 mm to (300.0, 55.6)
- moved POGO3 5.56 mm to (330.2, 55.6)
- moved POGO4 5.56 mm to (404.8, 55.6)
Routing:
- net VCC: track 466.1 -> 440.0 mm, vias 4 -> 3
- net GND: track 441.0 -> 416.6 mm, vias 2 -> 0
- net SERIAL: track 468.3 -> 445.1 mm, vias 0 -> 1
Other:
- board size 423.9 x 98.4 mm -> 412.8 x 98.4 mm
- net class Default removed
- net class Power removed
