File: 65NumpadPLATE.kicad_pcb (KiCad board)
At the start: 2 copper layers, 565 x 98.6 mm, 65 parts

Commit message: Forgot the solder mask :(
Other:
- net class Default removed
- net class Power removed
